Commit message: add camera joint to urdf

File: src/my_first_package/urdf/simple_mobile_robot.urdf (robot description, URDF)
Before this commit: robot simple_mobile_robot, 6 links, 5 joints
Links:
- added link camera_link; visual box size=0.04 0.04 0.03
Joints:
- added joint camera_joint: type fixed, parent base_link, child camera_link, origin xyz=0.16 0.0 0.12 rpy=0.0 0.0 0.0
